Commit message: add collision and inertial params for gazebo sim. Implement correct sim cams

File: urdf/zed.urdf.xacro (robot description, xacro)
@@ -19,4 +19,5 @@
     <xacro:include filename="$(find zed_description)/urdf/materials.urdf.xacro" />
     <!-- Arguments -->
+    <xacro:arg name="tf_prefix"     default="" />
     <xacro:arg name="camera_name"   default="zed" />
     <xacro:arg name="camera_model"  default="zed" />
@@ -56,4 +57,14 @@
             <material name="${model}_mat" />
         </visual>
+        <collision>
+            <origin xyz="0 0 0" rpy="0 0 0"/>
+            <geometry>
+                <mesh filename="package://zed_description/meshes/${model}.stl" />
+            </geometry>
+        </collision>
+        <inertial>
+            <mass value=".135" />
+            <inertia ixx="1.0" ixy="0.0" ixz="0.0" iyy="1.0" iyz="0.0" izz="1.0" />
+        </inertial>
     </link>
 <!-- Left Camera -->
@@ -110,3 +121,4 @@
         <link name="$(arg camera_name)_temp_right_link" />
     </xacro:if>
+    <xacro:include filename="$(find zed_description)/urdf/zed.gazebo" />
 </robot>
